Commit message: update

File: multi_mir_robot_description/urdf/include/mir_100_v1.urdf.xacro (robot description, xacro)
@@ -3,5 +3,5 @@
   <xacro:arg name="prefix" default=""/>
   <xacro:arg name="mir_type" default="mir_100"/>
-  <xacro:include filename="$(find mir_description)/urdf/include/mir_v1.urdf.xacro" />
+  <xacro:include filename="$(find multi_mir_robot_description)/urdf/include/mir_v1.urdf.xacro" />
   <xacro:mir prefix="${prefix}" />
 </robot>

File: multi_mir_robot_description/urdf/include/mir_v1.urdf.xacro (robot description, xacro)
@@ -3,9 +3,9 @@
   <xacro:arg name="mir_type" default="mir_100" />      <!-- The MiR variant. Can be "mir_100" or "mir_250" for now.-->
   <xacro:property name="mir_type" value="$(arg mir_type)" />  <!-- necessary because args cannot be accessed inside ${} expressions -->
-  <xacro:include filename="$(find mir_description)/urdf/include/common_properties.urdf.xacro" />
-  <xacro:include filename="$(find mir_description)/urdf/include/imu.gazebo.urdf.xacro" />
-  <xacro:include filename="$(find mir_description)/urdf/include/mir.gazebo.xacro" />
-  <xacro:include filename="$(find mir_description)/urdf/include/mir.transmission.xacro" />
-  <xacro:include filename="$(find mir_description)/urdf/include/sick_s300.urdf.xacro" />
+  <xacro:include filename="$(find multi_mir_robot_description)/urdf/include/common_properties.urdf.xacro" />
+  <xacro:include filename="$(find multi_mir_robot_description)/urdf/include/imu.gazebo.urdf.xacro" />
+  <xacro:include filename="$(find multi_mir_robot_description)/urdf/include/mir.gazebo.xacro" />
+  <xacro:include filename="$(find multi_mir_robot_description)/urdf/include/mir.transmission.xacro" />
+  <xacro:include filename="$(find multi_mir_robot_description)/urdf/include/sick_s300.urdf.xacro" />
   <xacro:property name="deg_to_rad" value="0.017453293" />
   <!-- The inertia for the MiR platform is intentionally chosen to be smaller than
@@ -115,5 +115,5 @@
         <origin xyz="0 0 0" rpy="0 0 0" />
         <geometry>
-          <mesh filename="package://mir_description/meshes/visual/caster_wheel_base.stl" />
+          <mesh filename="package://multi_mir_robot_description/meshes/visual/caster_wheel_base.stl" />
         </geometry>
         <xacro:if value="${mir_type == 'mir_100'}">
@@ -127,5 +127,5 @@
         <origin xyz="0 0 0" rpy="0 0 0" />
         <geometry>
-          <mesh filename="package://mir_description/meshes/collision/caster_wheel_base.stl" />
+          <mesh filename="package://multi_mir_robot_description/meshes/collision/caster_wheel_base.stl" />
         </geometry>
       </collision>
@@ -182,5 +182,5 @@
         <origin xyz="${mir_act_wheel_dx} 0 0" rpy="0 0 0" />
         <geometry>
-          <mesh filename="package://mir_description/meshes/visual/${mir_type}_base.stl" />
+          <mesh filename="package://multi_mir_robot_description/meshes/visual/${mir_type}_base.stl" />
         </geometry>
         <xacro:if value="${mir_type == 'mir_100'}">
@@ -194,5 +194,5 @@
         <origin xyz="${mir_act_wheel_dx} 0 0" rpy="0 0 0" />
         <geometry>
-          <mesh filename="package://mir_description/meshes/collision/${mir_type}_base.stl" />
+          <mesh filename="package://multi_mir_robot_description/meshes/collision/${mir_type}_base.stl" />
         </geometry>
       </collision>

File: multi_mir_robot_description/urdf/include/sick_s300.urdf.xacro (robot description, xacro)
@@ -1,5 +1,5 @@
 <?xml version="1.0"?>
 <robot xmlns:xacro="http://ros.org/wiki/xacro">
-  <xacro:include filename="$(find mir_description)/urdf/include/common_properties.urdf.xacro" />
+  <xacro:include filename="$(find multi_mir_robot_description)/urdf/include/common_properties.urdf.xacro" />
   <xacro:property name="laser_x" value="0.156" />
   <xacro:property name="laser_y" value="0.155" />
@@ -11,5 +11,5 @@
         <origin xyz="0.0 0.0 0.0" rpy="${pi} 0 0" />
         <geometry>
-          <mesh filename="package://mir_description/meshes/visual/sick_lms-100.stl" />
+          <mesh filename="package://multi_mir_robot_description/meshes/visual/sick_lms-100.stl" />
         </geometry>
         <!-- <xacro:insert_block name="material_yellow" /> -->
@@ -19,5 +19,5 @@
         <origin xyz="0.0 0.0 0.0" rpy="${pi} 0 0" />
         <geometry>
-          <mesh filename="package://mir_description/meshes/visual/sick_lms-100.stl" />
+          <mesh filename="package://multi_mir_robot_description/meshes/visual/sick_lms-100.stl" />
         </geometry>
       </collision>

File: multi_mir_robot_description/urdf/mir.urdf.xacro (robot description, xacro)
@@ -2,6 +2,6 @@
 <robot xmlns:xacro="http://ros.org/wiki/xacro" name="mir">
   <!-- MiR base -->
-  <xacro:include filename="$(find mir_description)/urdf/include/mir_v1.urdf.xacro" />
-  <xacro:include filename="$(find mir_description)/urdf/include/common.gazebo.xacro" />
+  <xacro:include filename="$(find multi_mir_robot_description)/urdf/include/mir_v1.urdf.xacro" />
+  <xacro:include filename="$(find multi_mir_robot_description)/urdf/include/common.gazebo.xacro" />
   <!-- Nhận prefix từ bên ngoài -->
   <xacro:arg name="prefix" default=""/>
